Commit message: Added robot_core2 URDF

File: description/gazebo_control.xacro (robot description, xacro)
@@ -1,20 +1,70 @@
 <?xml version="1.0"?>
 <robot xmlns:xacro="http://www.ros.org/wiki/xacro"  name="robot">
-    <gazebo>
-        <plugin name="diff_drive" filename="libgazebo_ros_diff_drive.so">
+    <!-- <gazebo>
+        <plugin name="diff_drive" filename="libgazebo_ros_diff_drive.so"> -->
             <!-- Wheel Information -->
-            <left_joint>left_wheel_joint</left_joint>
+            <!-- <left_joint>left_wheel_joint</left_joint>
             <right_joint>right_wheel_joint</right_joint>
             <wheel_separation>0.35</wheel_separation>
-            <wheel_diameter>0.1</wheel_diameter>
+            <wheel_diameter>0.1</wheel_diameter> -->
             <!-- Limits -->
-            <max_wheel_torque>200</max_wheel_torque>
+            <!-- <max_wheel_torque>200</max_wheel_torque>
+            <max_wheel_acceleration>10.0</max_wheel_acceleration> -->
+            <!-- Output -->
+            <!-- <odometry_frame>odom</odometry_frame>
+            <robot_base_frame>base_link</robot_base_frame> -->
+            <!-- <publish_odom>true</publish_odom>
+            <publish_odom_tf>true</publish_odom_tf>
+            <publish_wheel_tf>true</publish_wheel_tf>
+        </plugin> -->
+    <!-- </gazebo> -->
+    <!-- <gazebo>
+        <plugin name="skid_steer_drive_controller" filename="libgazebo_ros_diff_drive.so">
+             <updateRate>100.0</updateRate> -->
+            <!-- <robotNamespace>/</robotNamespace> -->
+            <!-- Wheel Information -->
+            <!-- <leftFrontJoint>left_front_wheel_joint</leftFrontJoint>
+            <rightFrontJoint>right_front_wheel_joint</rightFrontJoint>
+            <leftRearJoint>left_rear_wheel_joint</leftRearJoint>
+            <rightRearJoint>right_rear_wheel_joint</rightRearJoint> -->
+            <!-- Kinematics -->
+            <!-- <wheelSeparation>0.235</wheelSeparation>
+            <wheelDiameter>0.106</wheelDiameter>
+            <robotBaseFrame>chassis</robotBaseFrame> -->
+            <!-- Limits -->
+            <!-- <torque>11.8</torque>
             <max_wheel_acceleration>10.0</max_wheel_acceleration>
-            <!-- Output -->
+            <topicName>cmd_vel</topicName>
+            <broadcastTF>false</broadcastTF> -->
+        <!-- </plugin>
+    </gazebo>  -->
+     <gazebo>
+        <plugin name="diff_drive" filename="libgazebo_ros_diff_drive.so">
+            <!-- wheels -->
+            <num_wheel_pairs>2</num_wheel_pairs>
+            <left_joint>left_front_wheel_joint</left_joint>
+            <left_joint>left_rear_wheel_joint</left_joint>
+            <right_joint>right_front_wheel_joint</right_joint>
+            <right_joint>right_rear_wheel_joint</right_joint>
+            <!-- kinematics -->
+            <wheel_separation>0.235</wheel_separation>
+            <wheel_diameter>0.106</wheel_diameter>
+            <max_wheel_torque>11.8</max_wheel_torque>
+            <!-- <max_wheel_torque>200</max_wheel_torque>    -->
+            <max_wheel_acceleration>10.0</max_wheel_acceleration>
+            <!-- output  -->
+            <!-- <odometry_source>world</odometry_source> -->
             <odometry_frame>odom</odometry_frame>
-            <robot_base_frame>base_link</robot_base_frame>
+            <robot_base_frame>chassis</robot_base_frame>
+            <!-- topic & re remappings -->
+            <ros>
+                <namespace>/</namespace>
+                <argument>/cmd_vel:=cmd_vel</argument>
+                <argument>/odom:=odom</argument>
+            </ros>
             <publish_odom>true</publish_odom>
             <publish_odom_tf>true</publish_odom_tf>
             <publish_wheel_tf>true</publish_wheel_tf>
+            <!-- <update_rate>100.0</update_rate> -->
         </plugin>
     </gazebo>

File: description/robot.urdf.xacro (robot description, xacro)
@@ -2,5 +2,5 @@
 <robot xmlns:xacro="http://www.ros.org/wiki/xacro"  name="robot">
    <xacro:include filename="robot_core2.xacro"/>
-   <!-- <xacro:include filename="gazebo_control.xacro"/>
-   <xacro:include filename="lidar.xacro"/> -->
+   <xacro:include filename="gazebo_control.xacro"/>
+   <!-- <xacro:include filename="lidar.xacro"/> -->
 </robot>

File: description/robot_core2.xacro (robot description, xacro)
@@ -41,4 +41,7 @@
         </xacro:inertial_box>
     </link>
+    <gazebo reference="chassis">
+        <material>Gazebo/GreyTransparent</material>
+    </gazebo>
     <!-- LEFT FRONT WHEEL LINK -->
     <joint name="left_front_wheel_joint" type="continuous">
@@ -64,4 +67,9 @@
         </xacro:inertial_cylinder>
     </link>
+    <gazebo reference="left_front_wheel">
+        <material>Gazebo/Black</material>
+        <mu1 value="1"></mu1>
+        <mu2 value="0.8"></mu2>
+    </gazebo>
     <!-- LEFT REAR WHEEL LINK -->
     <joint name="left_rear_wheel_joint" type="continuous">
@@ -69,5 +77,5 @@
         <child link="left_rear_wheel"/>
         <origin xyz="-0.14 0.1175 -0.02" rpy="-${pi/2} 0 0" />
-        <axis xyz="0 0 -1"/>
+        <axis xyz="0 0 1"/>
     </joint>
     <link name="left_rear_wheel">
@@ -87,4 +95,9 @@
         </xacro:inertial_cylinder>
     </link>
+    <gazebo reference="left_rear_wheel">
+        <material>Gazebo/Black</material>
+        <mu1 value="1"></mu1>
+        <mu2 value="0.8"></mu2>
+    </gazebo>
     <!-- RIGHT FRONT WHEEL LINK -->
     <joint name="right_front_wheel_joint" type="continuous">
@@ -93,5 +106,5 @@
         <origin xyz="0.14 -0.1175 -0.02" rpy="
         ${pi/2} 0 0" />
-        <axis xyz="0 0 1"/>
+        <axis xyz="0 0 -1"/>
     </joint>
     <link name="right_front_wheel">
@@ -111,4 +124,9 @@
         </xacro:inertial_cylinder>
     </link>
+    <gazebo reference="right_front_wheel">
+        <material>Gazebo/Black</material>
+        <mu1 value="1"></mu1>
+        <mu2 value="0.8"></mu2>
+    </gazebo>
     <!-- RIGHT REAR WHEEL LINK -->
     <joint name="right_rear_wheel_joint" type="continuous">
@@ -134,3 +152,8 @@
         </xacro:inertial_cylinder>
     </link>
+    <gazebo reference="right_rear_wheel">
+        <material>Gazebo/Black</material>
+        <mu1 value="1"></mu1>
+        <mu2 value="0.8"></mu2>
+    </gazebo>
 </robot>

Commit message: URDF done

File: description/gazebo_control.xacro (robot description, xacro)
@@ -39,5 +39,5 @@
         <!-- </plugin>
     </gazebo>  -->
-     <gazebo>
+    <gazebo>
         <plugin name="diff_drive" filename="libgazebo_ros_diff_drive.so">
             <!-- wheels -->
@@ -49,10 +49,11 @@
             <!-- kinematics -->
             <wheel_separation>0.235</wheel_separation>
-            <wheel_diameter>0.106</wheel_diameter>
-            <max_wheel_torque>11.8</max_wheel_torque>
+            <wheel_diameter>0.1</wheel_diameter>
+            <max_wheel_torque>1.47</max_wheel_torque>
             <!-- <max_wheel_torque>200</max_wheel_torque>    -->
             <max_wheel_acceleration>10.0</max_wheel_acceleration>
             <!-- output  -->
             <!-- <odometry_source>world</odometry_source> -->
+            <odometry_source>1</odometry_source>
             <odometry_frame>odom</odometry_frame>
             <robot_base_frame>chassis</robot_base_frame>
@@ -66,5 +67,5 @@
             <publish_odom_tf>true</publish_odom_tf>
             <publish_wheel_tf>true</publish_wheel_tf>
-            <!-- <update_rate>100.0</update_rate> -->
+            <update_rate>100.0</update_rate>
         </plugin>
     </gazebo>

File: description/robot.urdf.xacro (robot description, xacro)
@@ -2,5 +2,5 @@
 <robot xmlns:xacro="http://www.ros.org/wiki/xacro"  name="robot">
    <xacro:include filename="robot_core2.xacro"/>
-   <xacro:include filename="gazebo_control.xacro"/>
+   <xacro:include filename="gazebo_control2.xacro"/>
    <!-- <xacro:include filename="lidar.xacro"/> -->
 </robot>

File: description/robot_core2.xacro (robot description, xacro)
@@ -38,5 +38,5 @@
         </collision>
         <xacro:inertial_box mass="0.5" x="0.4" y="0.18" z="0.005">
-            <origin xyz="0 0 0.07" rpy="0.0 0.0 0.0"/>
+            <origin xyz="0 0 0" rpy="0.0 0.0 0.0"/>
         </xacro:inertial_box>
     </link>
@@ -54,5 +54,5 @@
         <visual>
             <geometry>
-                <cylinder radius="0.053" length="0.044"/>
+                <cylinder radius="0.05" length="0.045"/>
             </geometry>
             <material name="black"/>
@@ -60,8 +60,8 @@
         <collision>
             <geometry>
-                <cylinder radius="0.053" length="0.044"/>
+                <cylinder radius="0.05" length="0.045"/>
             </geometry>
         </collision>
-        <xacro:inertial_cylinder mass="0.1" length="0.044" radius="0.053">
+        <xacro:inertial_cylinder mass="0.1" length="0.045" radius="0.05">
             <origin xyz="0 0 0" rpy="0.0 0.0 0.0"/>
         </xacro:inertial_cylinder>
@@ -69,6 +69,8 @@
     <gazebo reference="left_front_wheel">
         <material>Gazebo/Black</material>
-        <mu1 value="1"></mu1>
-        <mu2 value="0.8"></mu2>
+        <mu1 value="10"></mu1>
+        <mu2 value="10"></mu2>
+        <kp>1e10</kp>
+        <kd>1e8</kd>
     </gazebo>
     <!-- LEFT REAR WHEEL LINK -->
@@ -82,5 +84,5 @@
         <visual>
             <geometry>
-                <cylinder radius="0.053" length="0.044"/>
+                <cylinder radius="0.05" length="0.045"/>
             </geometry>
             <material name="black"/>
@@ -88,8 +90,8 @@
         <collision>
             <geometry>
-                <cylinder radius="0.053" length="0.044"/>
+                <cylinder radius="0.05" length="0.045"/>
             </geometry>
         </collision>
-        <xacro:inertial_cylinder mass="0.1" length="0.044" radius="0.053">
+        <xacro:inertial_cylinder mass="0.1" length="0.045" radius="0.05">
             <origin xyz="0 0 0" rpy="0.0 0.0 0.0"/>
         </xacro:inertial_cylinder>
@@ -97,6 +99,8 @@
     <gazebo reference="left_rear_wheel">
         <material>Gazebo/Black</material>
-        <mu1 value="1"></mu1>
-        <mu2 value="0.8"></mu2>
+        <mu1 value="10"></mu1>
+        <mu2 value="10"></mu2>
+        <kp>1e10</kp>
+        <kd>1e8</kd>
     </gazebo>
     <!-- RIGHT FRONT WHEEL LINK -->
@@ -111,5 +115,5 @@
         <visual>
             <geometry>
-                <cylinder radius="0.053" length="0.044"/>
+                <cylinder radius="0.05" length="0.045"/>
             </geometry>
             <material name="black"/>
@@ -117,8 +121,8 @@
         <collision>
             <geometry>
-                <cylinder radius="0.053" length="0.044"/>
+                <cylinder radius="0.05" length="0.045"/>
             </geometry>
         </collision>
-        <xacro:inertial_cylinder mass="0.1" length="0.044" radius="0.053">
+        <xacro:inertial_cylinder mass="0.1" length="0.045" radius="0.05">
             <origin xyz="0 0 0" rpy="0.0 0.0 0.0"/>
         </xacro:inertial_cylinder>
@@ -126,6 +130,8 @@
     <gazebo reference="right_front_wheel">
         <material>Gazebo/Black</material>
-        <mu1 value="1"></mu1>
-        <mu2 value="0.8"></mu2>
+        <mu1 value="10"></mu1>
+        <mu2 value="10"></mu2>
+        <kp>1e10</kp>
+        <kd>1e8</kd>
     </gazebo>
     <!-- RIGHT REAR WHEEL LINK -->
@@ -139,5 +145,5 @@
         <visual>
             <geometry>
-                <cylinder radius="0.053" length="0.044"/>
+                <cylinder radius="0.05" length="0.045"/>
             </geometry>
             <material name="black"/>
@@ -145,8 +151,8 @@
         <collision>
             <geometry>
-                <cylinder radius="0.053" length="0.044"/>
+                <cylinder radius="0.05" length="0.045"/>
             </geometry>
         </collision>
-        <xacro:inertial_cylinder mass="0.1" length="0.044" radius="0.053">
+        <xacro:inertial_cylinder mass="0.1" length="0.045" radius="0.05">
             <origin xyz="0 0 0" rpy="0.0 0.0 0.0"/>
         </xacro:inertial_cylinder>
@@ -154,6 +160,8 @@
     <gazebo reference="right_rear_wheel">
         <material>Gazebo/Black</material>
-        <mu1 value="1"></mu1>
-        <mu2 value="0.8"></mu2>
+        <mu1 value="10"></mu1>
+        <mu2 value="10"></mu2>
+        <kp>1e10</kp>
+        <kd>1e8</kd>
     </gazebo>
 </robot>
