Commit message: Added maps

File: description/lidar2.xacro (robot description, xacro)
@@ -2,5 +2,6 @@
 <robot xmlns:xacro="http://www.ros.org/wiki/xacro"  name="robot">
     <joint name="laser_joint" type="fixed">
-        <parent link="chassis"/>
+        <!-- changed chassis to base_link below -->
+        <parent link="base_link"/>
         <child link="laser_frame"/>
         <origin xyz="0.07 0 0.023" rpy="0 0 0"/>

File: description/robot.urdf.xacro (robot description, xacro)
@@ -4,4 +4,4 @@
    <xacro:include filename="gazebo_control2.xacro"/>
    <xacro:include filename="lidar2.xacro"/>
-   <xacro:include filename="depth_camera.xacro"/>
+   <xacro:include filename="camera.xacro"/>
 </robot>

File: description/robot_core2.xacro (robot description, xacro)
@@ -24,5 +24,5 @@
         <parent link="base_link"/>
         <child link="base_footprint"/>
-        <origin xyz="0 0 -0.07" rpy="0 0 0"/>
+        <origin xyz="0 0 0" rpy="0 0 0"/>
     </joint>
     <link name="base_footprint">
