Commit message: Added LiDar urdf

File: description/robot.urdf.xacro (robot description, xacro)
@@ -2,3 +2,5 @@
 <robot xmlns:xacro="http://www.ros.org/wiki/xacro"  name="robot">
    <xacro:include filename="robot_core.xacro"/>
+   <xacro:include filename="gazebo_control.xacro"/>
+   <xacro:include filename="lidar.xacro"/>
 </robot>

File: description/robot_core.xacro (robot description, xacro)
@@ -1,5 +1,5 @@
 <?xml version="1.0"?>
 <robot xmlns:xacro="http://www.ros.org/wiki/xacro"  >
-    <xacro:include filename="inertial_maxros.xacro"/>
+    <xacro:include filename="inertial_macros.xacro"/>
    <material name="white">
        <color rgba="1 1 1 1"/>
@@ -14,4 +14,7 @@
        <color rgba="0 0 0 1" />
    </material>
+    <material name="red">
+        <color rgba="1 0 0 1" />
+    </material>
    <!-- BASE LINK -->
    <link name="base_link">
@@ -41,4 +44,7 @@
        </xacro:inertial_box>
    </link>
+   <gazebo reference="chassis">
+        <material>Gazebo/White</material>
+   </gazebo>
    <!--  LEFT WHEEL -->
    <joint name="left_wheel_joint" type="continuous">
@@ -64,4 +70,7 @@
        </xacro:inertial_cylinder>
    </link>
+    <gazebo reference="left_wheel">
+        <material>Gazebo/Blue</material>
+    </gazebo>
    <!--  RIGHT WHEEL -->
    <joint name="right_wheel_joint" type="continuous">
@@ -87,4 +96,7 @@
         </xacro:inertial_cylinder>
     </link>
+    <gazebo reference="right_wheel">
+        <material>Gazebo/Blue</material>
+    </gazebo>
     <!-- CASTOR WHEEL LINK -->
     <joint name="castor_wheel_joint" type="fixed">
@@ -109,3 +121,8 @@
         </xacro:inertial_sphere>
     </link>
+    <gazebo reference="castor_wheel">
+        <material>Gazebo/Black</material>
+        <mu1 value="0.001"/>
+        <mu2 value="0.001"/>
+    </gazebo>
 </robot>

Commit message: added depth

File: description/robot.urdf.xacro (robot description, xacro)
@@ -3,4 +3,5 @@
    <xacro:include filename="robot_core2.xacro"/>
    <xacro:include filename="gazebo_control2.xacro"/>
-   <xacro:include filename="camera.xacro"/>
+   <xacro:include filename="lidar2.xacro"/>
+   <xacro:include filename="depth_camera.xacro"/>
 </robot>

File: description/robot_core2.xacro (robot description, xacro)
@@ -19,4 +19,12 @@
     <!-- BASE LINK -->
     <link name="base_link">
+    </link>
+    <!-- BASE_FOOTPRINT LINK -->
+    <joint name="base_footprint_joint" type="fixed">
+        <parent link="base_link"/>
+        <child link="base_footprint"/>
+        <origin xyz="0 0 -0.07" rpy="0 0 0"/>
+    </joint>
+    <link name="base_footprint">
     </link>
     <!-- CHASSIS LINK -->

Commit message: added ros2_control extra bits

File: description/robot.urdf.xacro (robot description, xacro)
@@ -1,7 +1,12 @@
 <?xml version="1.0"?>
 <robot xmlns:xacro="http://www.ros.org/wiki/xacro"  name="robot">
+   <xacro:arg name="use_ros2_control" default="true"/>
    <xacro:include filename="robot_core2.xacro"/>
-   <!-- <xacro:include filename="gazebo_control2.xacro"/> -->
-   <xacro:include filename="ros2_control.xacro"/>
+   <xacro:if value="$(arg use_ros2_control)">
+      <xacro:include filename="ros2_control.xacro" />
+   </xacro:if>
+   <xacro:unless value="$(arg use_ros2_control)">
+      <xacro:include filename="gazebo_control2.xacro" />
+   </xacro:unless>
    <xacro:include filename="lidar2.xacro"/>
    <!-- <xacro:include filename="camera.xacro"/> -->

File: description/robot_core.xacro (robot description, xacro)
@@ -63,5 +63,5 @@
        <collision>
         <geometry>
-            <cylinder radius="0.05" length="0.04"/>
+            <sphere radius="0.05"/>
         </geometry>
        </collision>
@@ -89,5 +89,5 @@
         <collision>
             <geometry>
-                <cylinder radius="0.05" length="0.04"/>
+                <sphere radius="0.05"/>
             </geometry>
         </collision>

File: description/robot_core2.xacro (robot description, xacro)
@@ -71,5 +71,5 @@
         <collision>
             <geometry>
-                <cylinder radius="0.05" length="0.045"/>
+                <sphere radius="0.05"/>
             </geometry>
         </collision>
@@ -101,5 +101,5 @@
         <collision>
             <geometry>
-                <cylinder radius="0.05" length="0.045"/>
+                <sphere radius="0.05"/>
             </geometry>
         </collision>
@@ -132,5 +132,5 @@
         <collision>
             <geometry>
-                <cylinder radius="0.05" length="0.045"/>
+                <sphere radius="0.05"/>
             </geometry>
         </collision>
@@ -162,5 +162,5 @@
         <collision>
             <geometry>
-                <cylinder radius="0.05" length="0.045"/>
+                <sphere radius="0.05"/>
             </geometry>
         </collision>

File: description/ros2_control.xacro (robot description, xacro)
@@ -15,6 +15,6 @@
     <joint name="left_rear_wheel_joint">
       <command_interface name="velocity">
-        <param name="min">-10</param>
-        <param name="max">10</param>
+        <param name="min">-100</param>
+        <param name="max">100</param>
       </command_interface>
       <state_interface name="velocity"/>
@@ -23,6 +23,6 @@
     <joint name="right_front_wheel_joint">
       <command_interface name="velocity">
-        <param name="min">-10</param>
-        <param name="max">10</param>
+        <param name="min">-100</param>
+        <param name="max">100</param>
       </command_interface>
       <state_interface name="velocity"/>
@@ -31,6 +31,6 @@
     <joint name="right_rear_wheel_joint">
       <command_interface name="velocity">
-        <param name="min">-10</param>
-        <param name="max">10</param>
+        <param name="min">-100</param>
+        <param name="max">100</param>
       </command_interface>
       <state_interface name="velocity"/>
