Commit message: Added camera XACRO

File: description/gazebo_control2.xacro (robot description, xacro)
@@ -32,6 +32,6 @@
         <publish_odom_tf>true</publish_odom_tf>
         <publish_wheel_tf>true</publish_wheel_tf>
-        <odometry_frame>base_link</odometry_frame>
-        <robot_base_frame>chassis</robot_base_frame>
+        <odometry_frame>odom</odometry_frame>
+        <robot_base_frame>base_link</robot_base_frame>
       </plugin>
     </gazebo>

File: description/robot.urdf.xacro (robot description, xacro)
@@ -3,4 +3,4 @@
    <xacro:include filename="robot_core2.xacro"/>
    <xacro:include filename="gazebo_control2.xacro"/>
-   <!-- <xacro:include filename="lidar.xacro"/> -->
+   <xacro:include filename="camera.xacro"/>
 </robot>

File: description/robot_core2.xacro (robot description, xacro)
@@ -14,4 +14,7 @@
         <color rgba="0 0 0 1"/>
     </material>
+    <material name="red">
+        <color rgba="1 0 0 1"/>
+    </material>
     <!-- BASE LINK -->
     <link name="base_link">
@@ -21,9 +24,9 @@
         <parent link="base_link"/>
         <child link="chassis"/>
-        <origin xyz="0 0 0.07"/>
+        <origin xyz="0 0 0"/>
     </joint>
     <link name="chassis">
         <visual>
-            <!-- <origin xyz="0 0 0.07"/> -->
+            <origin xyz="0 0 0"/>
             <geometry>
                 <box size="0.4 0.18 0.005"/>
@@ -32,5 +35,5 @@
         </visual>
         <collision>
-            <!-- <origin xyz="0 0 0.07"/> -->
+            <origin xyz="0 0 0"/>
             <geometry>
                 <box size="0.4 0.18 0.005"/>
@@ -46,5 +49,5 @@
     <!-- LEFT FRONT WHEEL LINK -->
     <joint name="left_front_wheel_joint" type="continuous">
-        <parent link="chassis"/>
+        <parent link="base_link"/>
         <child link="left_front_wheel"/>
         <origin xyz="0.14 0.1175 -0.02" rpy="-${pi/2} 0 0" />
@@ -76,5 +79,5 @@
     <!-- LEFT REAR WHEEL LINK -->
     <joint name="left_rear_wheel_joint" type="continuous">
-        <parent link="chassis"/>
+        <parent link="base_link"/>
         <child link="left_rear_wheel"/>
         <origin xyz="-0.14 0.1175 -0.02" rpy="-${pi/2} 0 0" />
@@ -106,5 +109,5 @@
     <!-- RIGHT FRONT WHEEL LINK -->
     <joint name="right_front_wheel_joint" type="continuous">
-        <parent link="chassis"/>
+        <parent link="base_link"/>
         <child link="right_front_wheel"/>
         <origin xyz="0.14 -0.1175 -0.02" rpy="
@@ -137,5 +140,5 @@
     <!-- RIGHT REAR WHEEL LINK -->
     <joint name="right_rear_wheel_joint" type="continuous">
-        <parent link="chassis"/>
+        <parent link="base_link"/>
         <child link="right_rear_wheel"/>
         <origin xyz="-0.14 -0.1175 -0.02" rpy="${pi/2} 0 0" />

Commit message: fixed laser_frame

File: description/gazebo_control2.xacro (robot description, xacro)
@@ -15,9 +15,9 @@
         <num_wheel_pairs>2</num_wheel_pairs>
         <!-- wheels0 -->
-        <left_joint>left_front_wheel_joint</left_joint>
-        <right_joint>right_front_wheel_joint</right_joint>
+        <left_joint>front_left_wheel_joint</left_joint>
+        <right_joint>front_right_wheel_joint</right_joint>
         <!-- wheels1-->
-        <left_joint>left_rear_wheel_joint</left_joint>
-        <right_joint>right_rear_wheel_joint</right_joint>
+        <left_joint>rear_left_wheel_joint</left_joint>
+        <right_joint>rear_right_wheel_joint</right_joint>
         <!-- kinematics -->
         <wheel_separation>0.235</wheel_separation>

File: description/lidar2.xacro (robot description, xacro)
@@ -23,5 +23,5 @@
         </xacro:inertial_cylinder>
     </link>
-    <gazebo reference="laser_frame">
+    <!-- <gazebo reference="laser_frame">
         <material>Gazebo/Red</material>
         <sensor name="laser" type="ray">
@@ -52,4 +52,4 @@
             </plugin>
         </sensor>
-    </gazebo>
+    </gazebo> -->
 </robot>

File: description/robot_core2.xacro (robot description, xacro)
@@ -56,11 +56,11 @@
     </gazebo>
     <!-- LEFT FRONT WHEEL LINK -->
-    <joint name="left_front_wheel_joint" type="continuous">
+    <joint name="front_left_wheel_joint" type="continuous">
         <parent link="base_link"/>
-        <child link="left_front_wheel"/>
+        <child link="front_left_wheel"/>
         <origin xyz="0.14 0.1175 -0.02" rpy="-${pi/2} 0 0" />
         <axis xyz="0 0 1"/>
     </joint>
-    <link name="left_front_wheel">
+    <link name="front_left_wheel">
         <visual>
             <geometry>
@@ -78,5 +78,5 @@
         </xacro:inertial_cylinder>
     </link>
-    <gazebo reference="left_front_wheel">
+    <gazebo reference="front_left_wheel">
         <material>Gazebo/Black</material>
         <mu1 value="10"></mu1>
@@ -86,11 +86,11 @@
     </gazebo>
     <!-- LEFT REAR WHEEL LINK -->
-    <joint name="left_rear_wheel_joint" type="continuous">
+    <joint name="rear_left_wheel_joint" type="continuous">
         <parent link="base_link"/>
-        <child link="left_rear_wheel"/>
+        <child link="rear_left_wheel"/>
         <origin xyz="-0.14 0.1175 -0.02" rpy="-${pi/2} 0 0" />
         <axis xyz="0 0 1"/>
     </joint>
-    <link name="left_rear_wheel">
+    <link name="rear_left_wheel">
         <visual>
             <geometry>
@@ -108,5 +108,5 @@
         </xacro:inertial_cylinder>
     </link>
-    <gazebo reference="left_rear_wheel">
+    <gazebo reference="rear_left_wheel">
         <material>Gazebo/Black</material>
         <mu1 value="10"></mu1>
@@ -116,12 +116,12 @@
     </gazebo>
     <!-- RIGHT FRONT WHEEL LINK -->
-    <joint name="right_front_wheel_joint" type="continuous">
+    <joint name="front_right_wheel_joint" type="continuous">
         <parent link="base_link"/>
-        <child link="right_front_wheel"/>
+        <child link="front_right_wheel"/>
         <origin xyz="0.14 -0.1175 -0.02" rpy="
         ${pi/2} 0 0" />
         <axis xyz="0 0 -1"/>
     </joint>
-    <link name="right_front_wheel">
+    <link name="front_right_wheel">
         <visual>
             <geometry>
@@ -139,5 +139,5 @@
         </xacro:inertial_cylinder>
     </link>
-    <gazebo reference="right_front_wheel">
+    <gazebo reference="front_right_wheel">
         <material>Gazebo/Black</material>
         <mu1 value="10"></mu1>
@@ -147,11 +147,11 @@
     </gazebo>
     <!-- RIGHT REAR WHEEL LINK -->
-    <joint name="right_rear_wheel_joint" type="continuous">
+    <joint name="rear_right_wheel_joint" type="continuous">
         <parent link="base_link"/>
-        <child link="right_rear_wheel"/>
+        <child link="rear_right_wheel"/>
         <origin xyz="-0.14 -0.1175 -0.02" rpy="${pi/2} 0 0" />
         <axis xyz="0 0 -1"/>
     </joint>
-    <link name="right_rear_wheel">
+    <link name="rear_right_wheel">
         <visual>
             <geometry>
@@ -169,5 +169,5 @@
         </xacro:inertial_cylinder>
     </link>
-    <gazebo reference="right_rear_wheel">
+    <gazebo reference="rear_right_wheel">
         <material>Gazebo/Black</material>
         <mu1 value="10"></mu1>

File: description/ros2_control.xacro (robot description, xacro)
@@ -5,23 +5,15 @@
       <!-- <plugin>diffdrive_arduino/DiffDriveArduino</plugin> -->
       <plugin>ros2_control_demo_example_2/DiffBotSystemHardware</plugin>
-      <!-- <param name="left_wheel_name">left_front_wheel_joint</param> -->
-      <param name="left_wheel_name">left_rear_wheel_joint</param>
-      <!-- <param name="right_wheel_name">right_front_wheel_joint</param> -->
-      <param name="right_wheel_name">right_rear_wheel_joint</param>
+      <param name="left_wheel_name">front_left_wheel_joint</param>
+      <param name="left_wheel_name">rear_left_wheel_joint</param>
+      <param name="right_wheel_name">front_right_wheel_joint</param>
+      <param name="right_wheel_name">rear_right_wheel_joint</param>
       <param name="loop_rate">30</param>
-      <param name="device">/dev/ttyUSB0</param>
-      <param name="baud_rate">57600</param>
-      <param name="timeout">1000</param>
-      <param name="enc_counts_per_rev">540</param>
+      <!-- <param name="device">/dev/ttyUSB0</param> -->
+      <!-- <param name="baud_rate">57600</param> -->
+      <!-- <param name="timeout">1000</param> -->
+      <!-- <param name="enc_counts_per_rev">540</param> -->
     </hardware>
-    <joint name="left_front_wheel_joint">
-      <command_interface name="velocity">
-        <param name="min">-10</param>
-        <param name="max">10</param>
-      </command_interface>
-      <state_interface name="velocity"/>
-      <state_interface name="position"/>
-    </joint>
-    <joint name="left_rear_wheel_joint">
+    <joint name="front_left_wheel_joint">
       <command_interface name="velocity">
         <param name="min">-100</param>
@@ -31,5 +23,5 @@
       <state_interface name="position"/>
     </joint>
-    <joint name="right_front_wheel_joint">
+    <joint name="rear_left_wheel_joint">
       <command_interface name="velocity">
         <param name="min">-100</param>
@@ -39,5 +31,13 @@
       <state_interface name="position"/>
     </joint>
-    <joint name="right_rear_wheel_joint">
+    <joint name="front_right_wheel_joint">
+      <command_interface name="velocity">
+        <param name="min">-100</param>
+        <param name="max">100</param>
+      </command_interface>
+      <state_interface name="velocity"/>
+      <state_interface name="position"/>
+    </joint>
+    <joint name="rear_right_wheel_joint">
       <command_interface name="velocity">
         <param name="min">-100</param>
@@ -54,6 +54,6 @@
     <joint name="left_front_wheel_joint">
       <command_interface name="velocity">
-        <param name="min">-10</param>
-        <param name="max">10</param>
+        <param name="min">-100</param>
+        <param name="max">100</param>
       </command_interface>
       <state_interface name="velocity"/>

Commit message: changed wheel specs

File: description/gazebo_control2.xacro (robot description, xacro)
@@ -21,6 +21,6 @@
         <right_joint>rear_right_wheel_joint</right_joint>
         <!-- kinematics -->
-        <wheel_separation>0.235</wheel_separation>
-        <wheel_separation>0.235</wheel_separation>
+        <wheel_separation>0.2025</wheel_separation>
+        <wheel_separation>0.2025</wheel_separation>
         <wheel_diameter>0.1</wheel_diameter>
         <wheel_diameter>0.1</wheel_diameter>

File: description/robot_core2.xacro (robot description, xacro)
@@ -65,5 +65,5 @@
         <visual>
             <geometry>
-                <cylinder radius="0.05" length="0.045"/>
+                <cylinder radius="0.0325" length="0.045"/>
             </geometry>
             <material name="black"/>
@@ -71,8 +71,8 @@
         <collision>
             <geometry>
-                <sphere radius="0.05"/>
+                <sphere radius="0.0325"/>
             </geometry>
         </collision>
-        <xacro:inertial_cylinder mass="0.1" length="0.045" radius="0.05">
+        <xacro:inertial_cylinder mass="0.1" length="0.045" radius="0.0325">
             <origin xyz="0 0 0" rpy="0.0 0.0 0.0"/>
         </xacro:inertial_cylinder>
@@ -95,5 +95,5 @@
         <visual>
             <geometry>
-                <cylinder radius="0.05" length="0.045"/>
+                <cylinder radius="0.0325" length="0.045"/>
             </geometry>
             <material name="black"/>
@@ -101,8 +101,8 @@
         <collision>
             <geometry>
-                <sphere radius="0.05"/>
+                <sphere radius="0.0325"/>
             </geometry>
         </collision>
-        <xacro:inertial_cylinder mass="0.1" length="0.045" radius="0.05">
+        <xacro:inertial_cylinder mass="0.1" length="0.045" radius="0.0325">
             <origin xyz="0 0 0" rpy="0.0 0.0 0.0"/>
         </xacro:inertial_cylinder>
@@ -126,5 +126,5 @@
         <visual>
             <geometry>
-                <cylinder radius="0.05" length="0.045"/>
+                <cylinder radius="0.0325" length="0.045"/>
             </geometry>
             <material name="black"/>
@@ -132,8 +132,8 @@
         <collision>
             <geometry>
-                <sphere radius="0.05"/>
+                <sphere radius="0.0325"/>
             </geometry>
         </collision>
-        <xacro:inertial_cylinder mass="0.1" length="0.045" radius="0.05">
+        <xacro:inertial_cylinder mass="0.1" length="0.045" radius="0.0325">
             <origin xyz="0 0 0" rpy="0.0 0.0 0.0"/>
         </xacro:inertial_cylinder>
@@ -156,5 +156,5 @@
         <visual>
             <geometry>
-                <cylinder radius="0.05" length="0.045"/>
+                <cylinder radius="0.0325" length="0.045"/>
             </geometry>
             <material name="black"/>
@@ -162,8 +162,8 @@
         <collision>
             <geometry>
-                <sphere radius="0.05"/>
+                <sphere radius="0.0325"/>
             </geometry>
         </collision>
-        <xacro:inertial_cylinder mass="0.1" length="0.045" radius="0.05">
+        <xacro:inertial_cylinder mass="0.1" length="0.045" radius="0.0325">
             <origin xyz="0 0 0" rpy="0.0 0.0 0.0"/>
         </xacro:inertial_cylinder>
