Commit message: done

File: description/robot_core2.xacro (robot description, xacro)
@@ -17,14 +17,14 @@
         <color rgba="1 0 0 1"/>
     </material>
+    <!-- BASE_FOOTPRINT LINK -->
+    <link name="base_footprint">
+    </link>
+    <joint name="base_footprint_joint" type="fixed">
+        <parent link="base_footprint"/>
+        <child link="base_link"/>
+        <origin xyz="0 0 0" rpy="0 0 0"/>
+    </joint>
     <!-- BASE LINK -->
     <link name="base_link">
-    </link>
-    <!-- BASE_FOOTPRINT LINK -->
-    <joint name="base_footprint_joint" type="fixed">
-        <parent link="base_link"/>
-        <child link="base_footprint"/>
-        <origin xyz="0 0 0" rpy="0 0 0"/>
-    </joint>
-    <link name="base_footprint">
     </link>
     <!-- CHASSIS LINK -->
